File: Circuit V1.sch (EAGLE design)
At the start: 23 parts, among them IC1 L298, J2 AVR_SPI_PROG_3X2PTH, J4 POWER_JACK, J6 1X2-3.5MM, U1 ATMEGA328P_TQFP, Y1 16MHz

Commit message: take 2
needs traces added
Parts:
- removed C1: 0.1uF, SparkFun-Capacitors:0.1UF-KIT-EZ-50V-20%
- removed D4, D6, D7: (no value), diode:DIODE-D-5
- removed J3: (no value), SparkFun-Connectors:CONN_03
- removed J5: (no value), SparkFun-Connectors:CONN_06SILK_FEMALE_PTH
- removed J6: 1X2-3.5MM, adafruit:1X2-3.5MM
- removed R4: 1k, SparkFun-Resistors:RESISTORAXIAL-0.3-KIT
- added D1, D2, D3: (no value), diode:DIODE-DO214AA
- added INSIDE_BUTTON, INSIDE_OPEN_BUTTON, LIGHT_SENSOR, LOCK_PIN1, LOCK_PIN2, MOTOR, OUTSIDE_BUTTON, OUTSIDE_OPEN_BUTTON, POT, POTPOWER, RESETBUTTON: 1X2-3.5MM, adafruit:1X2-3.5MM
- added R5, R6, R7: 10k, rcl:R-US_M0805
- C2: value 0.1uF -> 10*10^-6; device SparkFun-Capacitors:0.1UF-KIT-EZ-50V-20% -> rcl:C-EUC0805; SPICEPREFIX (none) -> 10uF
- C3: device SparkFun-Capacitors:0.1UF-KIT-EZ-50V-20% -> rcl:C-EUC0805
- C4, C5: device rcl:C-US050-024X044 -> rcl:C-EUC0805
- D5: device diode:DIODE-D-5 -> diode:DIODE-DO214AA
- J1: device SparkFun-Connectors:CONN_01 -> pinhead:PINHD-1X6
- R1, R3: value 1k -> 10k; device SparkFun-Resistors:RESISTORAXIAL-0.3-KIT -> rcl:R-US_M0805
- R2: device SparkFun-Resistors:RESISTORAXIAL-0.3-KIT -> rcl:R-US_M0805
Connections:
- net ENA renamed ENA_PWM
- net N$22 renamed AREF
- removed net DTR: C1.1, J1.1
- removed net N$21: D4.A, D5.C, IC1.OUT1, J6.1
- removed net N$23: D6.A, D7.C, IC1.OUT2, J6.2
- removed net N$3: J3.3, U1.PC2(ADC2)
- removed net N$6: C1.2, J2.5, R2.1, U1.PC6(/RESET)
- removed net RESET: J5.4, R1.1, U1.PD6(AIN0)
- removed net VCC: J2.2
- new net OPEN_CLOSE_BUTTON: INSIDE_BUTTON.1, OUTSIDE_BUTTON.1, R1.1, U1.PB0(ICP)
- new net OUT1: D3.A, D5.C, IC1.OUT1, MOTOR.1
- new net OUT2: D1.C, D2.A, IC1.OUT2, MOTOR.2
- new net RESEET: J2.5, R2.1, RESETBUTTON.2, U1.PC6(/RESET)
- new net RXD: J1.3, U1.PD0(RXD)
- new net TXD: J1.2, U1.PD1(TXD)
- net +5V: now also J2.2, POTPOWER.1, R6.2, R7.2; no longer J5.5, R4.2
- net 12V: now also D2.C, D3.C; no longer D4.C, D6.C
- net CLOSE_SWITCH: now also INSIDE_OPEN_BUTTON.1, R6.1, U1.PD7(AIN1); no longer J5.3, U1.PD5(T1)
- net GND: now also D1.A, IC1.ENABLE_B, IC1.INPUT3, IC1.INPUT4, INSIDE_BUTTON.2, INSIDE_OPEN_BUTTON.2, J1.6, LIGHT_SENSOR.2, LOCK_PIN1.2, LOCK_PIN2.2, OUTSIDE_BUTTON.2, OUTSIDE_OPEN_BUTTON.2, POT.2, POTPOWER.2, R5.2, RESETBUTTON.1; no longer D7.A, J5.6
- net LIGHT_SENSOR: now also LIGHT_SENSOR.1; no longer J3.1
- net LOCK_PIN: now also LOCK_PIN1.1, LOCK_PIN2.1, R5.1, U1.PD5(T1); no longer J5.1, U1.PD0(RXD)
- net OPEN_SWITCH: now also OUTSIDE_OPEN_BUTTON.1, R7.1, U1.PD6(AIN0); no longer J5.2, U1.PD1(TXD)
- net POT: now also POT.1; no longer J3.2, R4.1
Other:
- note added: "Connector for USB"
- note added: "Lock Pins"
- note added: "Open Close Buttons"
- note added: "Open close switches"
- note added: "Reset Button"
- note removed: "Open Close Button"
- note removed: "Reset button"
- moved on the sheet: C2, C4, R1, R2, R3
